Commit message: add force sensor

File: do_description/urdf/fourwheeler_base.urdf.xacro (robot description, xacro)
@@ -233,5 +233,7 @@
       </link>
       <!--hook for opening door-->
-      <joint name="joint_fbummer_hook" type="fixed">
+      <joint name="joint_fbummer_hook" type="revolute">
+        <axis xyz="0 1 0" rpy="0 0 0"/>
+        <limit velocity="0" effort="1000" lower="0" upper="0"/>
         <origin xyz="${bumper_x/2} -${bumper_y/2} ${bumper_z/2}" rpy="0 0 0"/>
         <parent link="link_fbumper"/>
@@ -254,5 +256,5 @@
           <mass value="${hook_m}"/>
           <origin rpy="0 0 0" xyz="0 0 0"/>
-          <inertia ixx="${1/12*hook_m*(hook_y*hook_y+hook_z*hook_z)}" ixy="0" ixz="0" iyy="${1/12*hook_m*(hook_z*hook_z+hook_x*hook_x)}" iyz="0" izz="${1/12*hook_m*(hook_x*hook_x+hook_y*hook_y)}"/>
+          <inertia ixx="${1/12*hook_m*(hook_y*hook_y+hook_z*hook_z)}" ixy="0" ixz="0" iyy="${1/12*hook_m*(hook_z*hook_z+4*hook_x*hook_x)}" iyz="0" izz="${1/12*hook_m*(4*hook_x*hook_x+hook_y*hook_y)}"/>
         </inertial>
       </link>
@@ -343,4 +345,20 @@
         <material>Gazebo/Black</material>
       </gazebo>
+      <!--ft force sensor in joint-->
+      <gazebo reference ="joint_fbummer_hook">
+        <provideFeedback>true</provideFeedback>
+      </gazebo>
+      <gazebo>
+        <plugin name="ft_sensor" filename="libgazebo_ros_ft_sensor.so">
+          <updateRate>100.0</updateRate>
+          <topicName>tf_sensor_topic</topicName>
+          <jointName>joint_fbummer_hook</jointName>
+          <noise>
+            <type>guassian</type>
+            <mean>0.0</mean>
+            <stddev>0.003</stddev>
+          </noise>
+        </plugin>
+      </gazebo>
     </xacro:macro>
 </robot>

Commit message: add more environment for testing

File: do_description/urdf/fourwheeler_base.urdf.xacro (robot description, xacro)
@@ -1,4 +1,5 @@
 <?xml version="1.0" ?>
 <robot xmlns:xacro="https://www.ros.org/wiki/xacro" >
+    <xacro:property name="friction" value="0.98"/>
     <xacro:property name="PI" value="3.1415926535897931"/>
     <xacro:property name="chassis_x" value="0.42" />
@@ -320,21 +321,21 @@
       </gazebo>
       <gazebo reference="link_lrwheel">
-        <mu1>0.98</mu1>
-        <mu2>0.98</mu2>
+        <mu1>${friction}</mu1>
+        <mu2>${friction}</mu2>
         <material>Gazebo/Black</material>
       </gazebo>
       <gazebo reference="link_rrwheel">
-        <mu1>0.98</mu1>
-        <mu2>0.98</mu2>
+        <mu1>${friction}</mu1>
+        <mu2>${friction}</mu2>
         <material>Gazebo/Black</material>
       </gazebo>
       <gazebo reference="link_lfwheel">
-        <mu1>0.98</mu1>
-        <mu2>0.98</mu2>
+        <mu1>${friction}</mu1>
+        <mu2>${friction}</mu2>
         <material>Gazebo/Black</material>
       </gazebo>
       <gazebo reference="link_rfwheel">
-        <mu1>0.98</mu1>
-        <mu2>0.98</mu2>
+        <mu1>${friction}</mu1>
+        <mu2>${friction}</mu2>
         <material>Gazebo/Black</material>
       </gazebo>

File: do_description/urdf/mobile_robot.urdf.xacro (robot description, xacro)
@@ -1,4 +1,5 @@
 <?xml version="1.0"?>
 <robot name="mobile_robot" xmlns:xacro="https://www.ros.org/wiki/xacro" >
+    <xacro:arg name="mu" default="0.98" />
     <xacro:property name="cam_support_x" value="0.05" />
     <xacro:property name="cam_support_y" value="0.05" />
@@ -7,4 +8,5 @@
     <!--mobile base-->
     <xacro:include filename="$(find do_description)/urdf/fourwheeler_base.urdf.xacro" />
+      <xacro:property name="friction" value="$(arg mu)"/>
     <xacro:fourwheeler_base_macro/>
     <!--camera support-->

Commit message: add test report

File: do_description/urdf/fourwheeler_base.urdf.xacro (robot description, xacro)
@@ -1,5 +1,6 @@
 <?xml version="1.0" ?>
 <robot xmlns:xacro="https://www.ros.org/wiki/xacro" >
-    <xacro:property name="friction" value="0.98"/>
+    <xacro:property name="friction_k" value="0.98"/>
+    <xacro:property name="friction_s" value="0.98"/>
     <xacro:property name="PI" value="3.1415926535897931"/>
     <xacro:property name="chassis_x" value="0.42" />
@@ -321,21 +322,21 @@
       </gazebo>
       <gazebo reference="link_lrwheel">
-        <mu1>${friction}</mu1>
-        <mu2>${friction}</mu2>
+        <mu1>${friction_k}</mu1>
+        <mu2>${friction_s}</mu2>
         <material>Gazebo/Black</material>
       </gazebo>
       <gazebo reference="link_rrwheel">
-        <mu1>${friction}</mu1>
-        <mu2>${friction}</mu2>
+        <mu1>${friction_k}</mu1>
+        <mu2>${friction_s}</mu2>
         <material>Gazebo/Black</material>
       </gazebo>
       <gazebo reference="link_lfwheel">
-        <mu1>${friction}</mu1>
-        <mu2>${friction}</mu2>
+        <mu1>${friction_k}</mu1>
+        <mu2>${friction_s}</mu2>
         <material>Gazebo/Black</material>
       </gazebo>
       <gazebo reference="link_rfwheel">
-        <mu1>${friction}</mu1>
-        <mu2>${friction}</mu2>
+        <mu1>${friction_k}</mu1>
+        <mu2>${friction_s}</mu2>
         <material>Gazebo/Black</material>
       </gazebo>

File: do_description/urdf/mobile_robot.urdf.xacro (robot description, xacro)
@@ -1,5 +1,6 @@
 <?xml version="1.0"?>
 <robot name="mobile_robot" xmlns:xacro="https://www.ros.org/wiki/xacro" >
-    <xacro:arg name="mu" default="0.98" />
+    <xacro:arg name="mu1" default="0.7" />
+    <xacro:arg name="mu2" default="0.98" />
     <xacro:property name="cam_support_x" value="0.05" />
     <xacro:property name="cam_support_y" value="0.05" />
@@ -8,5 +9,6 @@
     <!--mobile base-->
     <xacro:include filename="$(find do_description)/urdf/fourwheeler_base.urdf.xacro" />
-      <xacro:property name="friction" value="$(arg mu)"/>
+      <xacro:property name="friction_k" value="$(arg mu1)"/>
+      <xacro:property name="friction_s" value="$(arg mu2)"/>
     <xacro:fourwheeler_base_macro/>
     <!--camera support-->
