Commit message: add more test cases

File: do_description/urdf/fourwheeler_base_l.urdf.xacro (robot description, xacro)
@@ -238,5 +238,5 @@
         <axis xyz="0 1 0" rpy="0 0 0"/>
         <limit velocity="0" effort="1000" lower="0" upper="0"/>
-        <origin xyz="${bumper_x/2} -${bumper_y/2} ${bumper_z/2}" rpy="0 0 0"/>
+        <origin xyz="${bumper_x/2} ${bumper_y/2} ${bumper_z/2}" rpy="0 0 0"/>
         <parent link="link_fbumper"/>
         <child link="link_hook"/>
@@ -268,5 +268,5 @@
       <link name="link_tip">
         <visual>
-          <origin xyz="${tip_x/2} 0.02 ${tip_z/2}" rpy="0 0 0" />
+          <origin xyz="${tip_x/2} -0.02 ${tip_z/2}" rpy="0 0 0" />
           <geometry>
             <box size="${tip_x} ${tip_y} ${tip_z}"/>
@@ -274,5 +274,5 @@
         </visual>
         <collision>
-          <origin xyz="${tip_x/2} 0.02 ${tip_z/2}" rpy="0 0 0" />
+          <origin xyz="${tip_x/2} -0.02 ${tip_z/2}" rpy="0 0 0" />
           <geometry>
             <box size="${tip_x} ${tip_y} ${tip_z}"/>

File: do_description/urdf/mobile_robot.urdf.xacro (robot description, xacro)
@@ -1,5 +1,5 @@
 <?xml version="1.0"?>
 <robot name="mobile_robot" xmlns:xacro="https://www.ros.org/wiki/xacro" >
-    <xacro:arg name="mu1" default="0.7" />
+    <xacro:arg name="mu1" default="0.98" />
     <xacro:arg name="mu2" default="0.98" />
     <xacro:property name="cam_support_x" value="0.05" />
