Commit message: change style of plot

File: do_description/urdf/mobile_robot.urdf.xacro (robot description, xacro)
@@ -43,5 +43,5 @@
       <xacro:property name="location_y" value="0.0" />
       <xacro:property name="location_z" value="0.02" />
-      <xacro:property name="location_r" value="0" />
+      <xacro:property name="location_r" value="0.0" />
       <xacro:property name="location_p" value="-1.57" />
       <xacro:property name="location_y" value="0" />
